File: kicad/FlatPanelBoard/FlatPanelBoard/FlatPanelBoard.kicad_pcb (KiCad board)
At the start: 2 copper layers, 40.5 x 59.5 mm, 11 parts, among them J1 Power, J2 PWM, J3 LED+, J4 LED-, J5 Motor-, J6 Motor+, Q1 IRLZ44N

Commit message: Updated cad file and kicad to connect to pin 11 instead of pin 9
Connections:
- R1 pad 2: /*9 -> /*11
Routing:
- net /*11: track 0.00 -> 10.4 mm
- net /*9: track 9.26 -> 0.00 mm
Changed lines of the file:
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@@
 			(net "/*11")
 			(pinfunction "Pin_7_7")
-			(pintype "passive+no_connect")
+			(pintype "passive")
 		)
 		(pad "8" thru_hole circle
@@
 			(layers "*.Cu" "*.Mask")
 			(remove_unused_layers no)
-			(net "/*9")
+			(net "/*11")
 			(pintype "passive")
 		)
@@
 	)
 	(segment
-		(start 139.116 49.2)
-		(end 139.116 53.884)
+		(start 138 56.5)
+		(end 138 58)
 		(width 1)
 		(layer "F.Cu")
-		(net "/*9")
+		(net "/*11")
 	)
 	(segment
-		(start 139.116 53.884)
-		(end 138 55)
+		(start 134.036 49.2)
+		(end 134.036 52.536)
 		(width 1)
 		(layer "F.Cu")
-		(net "/*9")
+		(net "/*11")
 	)
 	(segment
-		(start 138 55)
-		(end 138 58)
+		(start 134.036 52.536)
+		(end 138 56.5)
 		(width 1)
 		(layer "F.Cu")
-		(net "/*9")
+		(net "/*11")
 	)
 	(segment
