File: kicad/FlatPanelBoard/FlatPanelBoard/FlatPanelBoard.kicad_sch (KiCad schematic)
At the start: 10 parts, among them J1 Power, J2 PWM, J3 LED+, J4 LED-, J5 Motor-, J6 Motor+, Q1 IRLZ44N

Commit message: Updated cad file and kicad to connect to pin 11 instead of pin 9
Connections:
- net *11: now also R1.2
- net *9: no longer R1.2
Changed lines of the file:
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@@
 		)
 	)
-	(label "*9"
+	(label "*11"
 		(at 109.22 30.48 0)
 		(effects
